File: HW_Tester/HW_Tester.kicad_sch (KiCad schematic)
At the start: 59 parts, among them J1 JTAG, J2 USB C Power, J3 011/030/040/05x, J4 001, J5 JDS USB, J6 SSD1306, J7 Boot Jumper, U1 STM32F303CBTx, U2 AMS1117-3.3, Y1 Crystal

Commit message: Completed board pending review
Parts:
- removed C1, C2: C, Capacitor_SMD:C_0603_1608Metric, symbol Device:C
- removed Y1: Crystal, Crystal:Resonator_SMD_Murata_CSTxExxV-3Pin_3.0x1.1mm, symbol Device:Crystal
- added Y1: (no value), symbol Device:Resonator
- TP1, TP10, TP11, TP12, TP13, TP14, TP15, TP16, TP17, TP18, TP19, TP2, TP20, TP21, TP22, TP23, TP24, TP25, TP26, TP27, TP28, TP29, TP3, TP30, TP31, TP32, TP33, TP34, TP4, TP5, TP6, TP7, TP8, TP9: value (none) -> TestPoint; footprint (none) -> TestPoint:TestPoint_Pad_D1.0mm
Connections:
- net GND: now also U1.8 (VSSA), Y1.2
- net R-: now reaches U1.6 (PF1)
- net R-: now also Y1.3
- net R+: now reaches U1.5 (PF0)
- net R+: now also Y1.1

Commit message: Updated placements, zones, and outline
Parts:
- Y1: value (none) -> Resonator; footprint (none) -> Crystal:Resonator_SMD_Murata_CSTxExxV-3Pin_3.0x1.1mm
Changed lines of the file:
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@@
       (effects (font (size 1.27 1.27)) hide)
     )
-    (property "Value" "" (id 1) (at 99.6951 46.7888 90)
+    (property "Value" "GND" (id 1) (at 99.6951 46.7888 90)
       (effects (font (size 1.27 1.27)) (justify right))
     )
@@
       (effects (font (size 1.27 1.27)) (justify left))
     )
-    (property "Value" "" (id 1) (at 110.7694 48.0572 90)
+    (property "Value" "Resonator" (id 1) (at 110.7694 48.0572 90)
       (effects (font (size 1.27 1.27)) (justify left))
     )
-    (property "Footprint" "" (id 2) (at 107.95 45.72 0)
+    (property "Footprint" "Crystal:Resonator_SMD_Murata_CSTxExxV-3Pin_3.0x1.1mm" (id 2) (at 107.95 45.72 0)
       (effects (font (size 1.27 1.27)) hide)
     )
